Commit message: 1

File: envs/model/quadruped/FullDoggo7.urdf (robot description, URDF)
Before this commit: robot FullDoggo2, 14 links, 13 joints
Links:
- removed link pip1
- removed link pip2
- removed link pip3
- removed link pip4
- removed link plane1
- removed link plane2
- removed link plane3
- removed link plane4
- removed link plane5
- added link a, mass 0.049612609423567; collision mesh filename=C:\Users\sq\Documents\full2\meshes\a.STL; visual mesh filename=C:\Users\sq\Documents\full2\meshes\a.STL
- added link b, mass 0.0946817219162806; collision mesh filename=C:\Users\sq\Documents\full2\meshes\b.STL; visual mesh filename=C:\Users\sq\Documents\full2\meshes\b.STL
- added link c, mass 0.0946817219162811; collision mesh filename=C:\Users\sq\Documents\full2\meshes\c.STL; visual mesh filename=C:\Users\sq\Documents\full2\meshes\c.STL
- added link d, mass 0.0514644320422948; collision mesh filename=C:\Users\sq\Documents\full2\meshes\d.STL; visual mesh filename=C:\Users\sq\Documents\full2\meshes\d.STL
- added link e, mass 0.0514644320423025; collision mesh filename=C:\Users\sq\Documents\full2\meshes\e.STL; visual mesh filename=C:\Users\sq\Documents\full2\meshes\e.STL
- added link f, mass 0.00607742634204188; collision mesh filename=C:\Users\sq\Documents\full2\meshes\f.STL; visual mesh filename=C:\Users\sq\Documents\full2\meshes\f.STL
- added link g, mass 0.011007632070168; collision mesh filename=C:\Users\sq\Documents\full2\meshes\g.STL; visual mesh filename=C:\Users\sq\Documents\full2\meshes\g.STL
- link base_link: mass 0.0496126113245419 -> 0.0628725; geometry collision mesh filename=C:\Users\sq\Documents\full2\meshes\base_link.STL; visual mesh filename=C:\Users\sq\Documents\full2\meshes\base_link.STL
- link hip11: mass 0.0178815824937254 -> 0.00662276690952864; geometry collision mesh filename=C:\Users\sq\Documents\full2\meshes\hip11.STL; visual mesh filename=C:\Users\sq\Documents\full2\meshes\hip11.STL
- link hip12: mass 0.0250306596643849 -> 0.00927126538729555; geometry collision mesh filename=C:\Users\sq\Documents\full2\meshes\hip12.STL; visual mesh filename=C:\Users\sq\Documents\full2\meshes\hip12.STL
- link knee11: mass 0.0304320456503251 -> 0.0304320456503239; geometry collision mesh filename=C:\Users\sq\Documents\full2\meshes\knee11.STL; visual mesh filename=C:\Users\sq\Documents\full2\meshes\knee11.STL
- link knee12: geometry collision mesh filename=C:\Users\sq\Documents\full2\meshes\knee12.STL; visual mesh filename=C:\Users\sq\Documents\full2\meshes\knee12.STL
Joints:
- removed joint pip1
- removed joint pip2
- removed joint pip3
- removed joint pip4
- removed joint plane1
- removed joint plane2
- removed joint plane3
- removed joint plane4
- removed joint plane5
- added joint a: type fixed, parent base_link, child a, origin xyz=-0.21 0.097160555546947 -0.016655813706978 rpy=-1.5707963267949 0 -1.5707963267949, axis 0 0 0
- added joint b: type fixed, parent base_link, child b, origin xyz=0.175 -0.097178593586223 -0.017010467191248 rpy=1.5707963267949 0.0523598775598271 1.5707963267949, axis 0 0 0
- added joint c: type fixed, parent base_link, child c, origin xyz=-0.175 0.097178593586224 -0.017 rpy=1.5707963267949 0.052359877559827 -1.5707963267949, axis 0 0 0
- added joint d: type fixed, parent base_link, child d, origin xyz=0.09 -9.98629534750042E-05 -0.068930142767599 rpy=1.5707963267949 0 1.5707963267949, axis 0 0 0
- added joint e: type fixed, parent base_link, child e, origin xyz=-0.09 9.98629534759958E-05 -0.068919675576351 rpy=-1.5707963267949 0 -1.5707963267949, axis 0 0 0
- added joint f: type fixed, parent base_link, child f, origin xyz=0.175 -0.107164888933769 -0.016487107628819 rpy=2.35619449019235 0.0523598775598078 1.57079632679492, axis 0 0 0
- added joint g: type fixed, parent base_link, child g, origin xyz=0.175 -0.11615255474656 -0.016016084022632 rpy=2.35619449019235 0.0523598775598309 1.5707963267949, axis 0 0 0
- joint hip11: axis 0 0 0 -> -1 0 0; origin xyz=-0.024292 0.00011102 -0.00011102 rpy=1.5708 0.55555 1.5708 -> xyz=-0.01405 0 0 rpy=-2.1263 0 0; parent pip1 -> g
- joint hip12: axis 0 0 0 -> -1 0 0; origin xyz=-0.013767 0.00011102 -0.00011102 rpy=-1.4018 1.5708 1.6655 -> xyz=-0.012525 0 0 rpy=0 0 0; parent pip1 -> f
- joint knee11: axis 0 0 0 -> -0.001857 0.013655 0.99991; origin xyz=0 0.09 0.010528 rpy=0 0 -1.5708 -> xyz=0.25029 0.39099 -0.1443 rpy=1.7779 -1.008 -1.7101
- joint knee12: axis 0 0 0 -> -0.008056 -0.015332 -0.99985; origin xyz=0 0.09 0.010525 rpy=-3.1416 0 1.5708 -> xyz=0.24691 -0.19066 -0.18039 rpy=-1.4282 -1.0136 1.5258
