Commit message: q

File: envs/model/quadruped/minitaur.urdf (robot description, URDF)
Before this commit: robot quadruped, 27 links, 26 joints
Links:
- link base_chassis_link: geometry collision box size=.17 0.10 .05; collision box size=.17 0.10 .05
- link motor_back_leftL_link: geometry collision cylinder length=0.026 radius=0.0434; visual mesh filename=tmotor3.obj scale=0.1 0.1 0.1
- link motor_back_leftR_link: geometry collision cylinder length=0.026 radius=0.0434; visual mesh filename=tmotor3.obj scale=0.1 0.1 0.1
- link motor_back_rightL_link: geometry collision cylinder length=0.026 radius=0.0434; visual mesh filename=tmotor3.obj scale=0.1 0.1 0.1
- link motor_back_rightR_link: geometry collision cylinder length=0.026 radius=0.0434; visual mesh filename=tmotor3.obj scale=0.1 0.1 0.1
- link motor_front_leftL_link: geometry collision cylinder length=0.026 radius=0.0434; visual mesh filename=tmotor3.obj scale=0.1 0.1 0.1
- link motor_front_leftR_link: geometry collision cylinder length=0.026 radius=0.0434; visual mesh filename=tmotor3.obj scale=0.1 0.1 0.1
- link motor_front_rightL_link: geometry collision cylinder length=0.026 radius=0.0434; visual mesh filename=tmotor3.obj scale=0.1 0.1 0.1
- link motor_front_rightR_link: geometry collision cylinder length=0.006 radius=0.002; visual mesh filename=tmotor3.obj scale=0.01 0.01 0.01
Joints:
- joint motor_back_leftL_joint: origin xyz=-0.21 0.025 0 rpy=1.57075 0 3.141592 -> xyz=-0.21 0.1 0 rpy=1.57075 0 3.141592
- joint motor_back_leftR_joint: origin xyz=-0.21 -0.04 0 rpy=1.57075 0 0 -> xyz=-0.21 0.035 0 rpy=1.57075 0 0
- joint motor_back_rightL_joint: origin xyz=-0.21 0.04 0 rpy=1.57075 0 3.141592 -> xyz=-0.21 -0.035 0 rpy=1.57075 0 3.141592
- joint motor_back_rightR_joint: origin xyz=-0.21 -0.025 0 rpy=1.57075 0 0 -> xyz=-0.21 -0.1 0 rpy=1.57075 0 0
- joint motor_front_leftL_joint: origin xyz=0.21 0.025 0 rpy=1.57075 0 3.141592 -> xyz=0.21 0.1 0 rpy=1.57075 0 3.141592
- joint motor_front_leftR_joint: origin xyz=0.21 -0.04 0 rpy=1.57075 0 0 -> xyz=0.21 0.035 0 rpy=1.57075 0 0
- joint motor_front_rightL_joint: origin xyz=0.21 0.04 0 rpy=1.57075 0 3.141592 -> xyz=0.21 -0.035 0 rpy=1.57075 0 3.141592
- joint motor_front_rightR_joint: origin xyz=0.21 -0.025 0 rpy=1.57075 0 0 -> xyz=0.21 -0.1 0 rpy=1.57075 0 0

Commit message: q

File: envs/model/quadruped/minitaur.urdf (robot description, URDF)
Before this commit: robot quadruped, 27 links, 26 joints
Links:
- link base_chassis_link: geometry collision box size=.17 0.10 .05; collision box size=.17 0.10 .05
